File: src/PCB/GIS.sch (KiCad schematic (older format))
At the start: 83 parts, among them J1 LED, J2 4PIN, J3 OLED, SW1 SW_PUSH, SW10 SW_PUSH, SW11 SW_PUSH, SW12 SW_PUSH, SW13 SW_PUSH, SW14 SW_PUSH, SW15 SW_PUSH, SW16 SW_PUSH, SW17 SW_PUSH, SW18 SW_PUSH, SW19 SW_PUSH, SW2 SW_PUSH, SW20 SW_PUSH, SW21 SW_PUSH, SW22 SW_PUSH, SW23 SW_PUSH, SW24 SW_PUSH, SW26 SW_PUSH, SW27 SW_PUSH, SW28 SW_PUSH, SW29 SW_PUSH, SW3 SW_PUSH, SW30 SW_PUSH, SW4 SW_PUSH, SW5 SW_PUSH, SW6 SW_PUSH, SW7 SW_PUSH, SW8 SW_PUSH, SW9 SW_PUSH, U1 ProMicro

Commit message: fixing diode hole size
Parts:
- D1, D10, D11, D12, D13, D14, D15, D16, D17, D18, D19, D2, D20, D21, D22, D23, D24, D26, D27, D28, D29, D3, D30, D4, D5, D6, D7, D8, D9: symbol SofleKeyboard-rescue:D-Lily58-cache-Lily58_Pro-rescue -> GIS-rescue:D-Lily58-cache-Lily58_Pro-rescue-SofleKeyboard-rescue
- J1: symbol SofleKeyboard-rescue:LED-Lily58-cache-Lily58_Pro-rescue -> GIS-rescue:LED-Lily58-cache-Lily58_Pro-rescue-SofleKeyboard-rescue
- J2: symbol SofleKeyboard-rescue:MJ-4PP-9-Lily58-cache-Lily58_Pro-rescue -> GIS-rescue:MJ-4PP-9-Lily58-cache-Lily58_Pro-rescue-SofleKeyboard-rescue
- J3: symbol SofleKeyboard-rescue:OLED-Lily58-cache-Lily58_Pro-rescue -> GIS-rescue:OLED-Lily58-cache-Lily58_Pro-rescue-SofleKeyboard-rescue
- R1, R2: symbol SofleKeyboard-rescue:R-Lily58-cache-Lily58_Pro-rescue -> GIS-rescue:R-Lily58-cache-Lily58_Pro-rescue-SofleKeyboard-rescue
- RSW1: symbol SofleKeyboard-rescue:SW_RST-Lily58-cache-Lily58_Pro-rescue -> GIS-rescue:SW_RST-Lily58-cache-Lily58_Pro-rescue-SofleKeyboard-rescue
- SW1, SW10, SW11, SW12, SW13, SW14, SW15, SW16, SW17, SW18, SW19, SW2, SW20, SW21, SW22, SW23, SW24, SW26, SW27, SW28, SW29, SW3, SW30, SW4, SW5, SW6, SW7, SW8, SW9: symbol SofleKeyboard-rescue:SW_PUSH-Lily58-cache-Lily58_Pro-rescue -> GIS-rescue:SW_PUSH-Lily58-cache-Lily58_Pro-rescue-SofleKeyboard-rescue
- TH1, TH2, TH3, TH4, TH5, TH6, TH7: symbol SofleKeyboard-rescue:HOLE-Lily58-cache-Lily58_Pro-rescue -> GIS-rescue:HOLE-Lily58-cache-Lily58_Pro-rescue-SofleKeyboard-rescue
- U1: symbol SofleKeyboard-rescue:ProMicro_2-Lily58-cache-Lily58_Pro-rescue -> GIS-rescue:ProMicro_2-Lily58-cache-Lily58_Pro-rescue-SofleKeyboard-rescue

Commit message: switching to better dual diode footprint
Parts:
- D1, D10, D11, D12, D13, D14, D15, D16, D17, D18, D19, D2, D20, D21, D22, D23, D24, D26, D27, D28, D29, D3, D30, D4, D5, D6, D7, D8, D9: footprint SofleKeyboard-footprint:Diode_SOD123 -> choc:D3_TH_SMD_v2
Changed lines of the file:
@@
 F 0 "D1" V 6146 2321 50  0000 R CNN
 F 1 "D" V 6055 2321 50  0000 R CNN
-F 2 "SofleKeyboard-footprint:Diode_SOD123" H 6100 2400 50  0001 C CNN
+F 2 "choc:D3_TH_SMD_v2" H 6100 2400 50  0001 C CNN
 F 3 "" H 6100 2400 50  0001 C CNN
 	1    6100 2400
@@
 F 0 "D2" V 6946 2321 50  0000 R CNN
 F 1 "D" V 6855 2321 50  0000 R CNN
-F 2 "SofleKeyboard-footprint:Diode_SOD123" H 6900 2400 50  0001 C CNN
+F 2 "choc:D3_TH_SMD_v2" H 6900 2400 50  0001 C CNN
 F 3 "" H 6900 2400 50  0001 C CNN
 	1    6900 2400
@@
 F 0 "D3" V 7746 2321 50  0000 R CNN
 F 1 "D" V 7655 2321 50  0000 R CNN
-F 2 "SofleKeyboard-footprint:Diode_SOD123" H 7700 2400 50  0001 C CNN
+F 2 "choc:D3_TH_SMD_v2" H 7700 2400 50  0001 C CNN
 F 3 "" H 7700 2400 50  0001 C CNN
 	1    7700 2400
@@
 F 0 "D4" V 8546 2321 50  0000 R CNN
 F 1 "D" V 8455 2321 50  0000 R CNN
-F 2 "SofleKeyboard-footprint:Diode_SOD123" H 8500 2400 50  0001 C CNN
+F 2 "choc:D3_TH_SMD_v2" H 8500 2400 50  0001 C CNN
 F 3 "" H 8500 2400 50  0001 C CNN
 	1    8500 2400
@@
 F 0 "D5" V 9346 2321 50  0000 R CNN
 F 1 "D" V 9255 2321 50  0000 R CNN
-F 2 "SofleKeyboard-footprint:Diode_SOD123" H 9300 2400 50  0001 C CNN
+F 2 "choc:D3_TH_SMD_v2" H 9300 2400 50  0001 C CNN
 F 3 "" H 9300 2400 50  0001 C CNN
 	1    9300 2400
@@
 F 0 "D6" V 10146 2321 50  0000 R CNN
 F 1 "D" V 10055 2321 50  0000 R CNN
-F 2 "SofleKeyboard-footprint:Diode_SOD123" H 10100 2400 50  0001 C CNN
+F 2 "choc:D3_TH_SMD_v2" H 10100 2400 50  0001 C CNN
 F 3 "" H 10100 2400 50  0001 C CNN
 	1    10100 2400
@@
 F 0 "D7" V 6146 2971 50  0000 R CNN
 F 1 "D" V 6055 2971 50  0000 R CNN
-F 2 "SofleKeyboard-footprint:Diode_SOD123" H 6100 3050 50  0001 C CNN
+F 2 "choc:D3_TH_SMD_v2" H 6100 3050 50  0001 C CNN
 F 3 "" H 6100 3050 50  0001 C CNN
 	1    6100 3050
@@
 F 0 "D8" V 6946 2971 50  0000 R CNN
 F 1 "D" V 6855 2971 50  0000 R CNN
-F 2 "SofleKeyboard-footprint:Diode_SOD123" H 6900 3050 50  0001 C CNN
+F 2 "choc:D3_TH_SMD_v2" H 6900 3050 50  0001 C CNN
 F 3 "" H 6900 3050 50  0001 C CNN
 	1    6900 3050
@@
 F 0 "D9" V 7746 2971 50  0000 R CNN
 F 1 "D" V 7655 2971 50  0000 R CNN
-F 2 "SofleKeyboard-footprint:Diode_SOD123" H 7700 3050 50  0001 C CNN
+F 2 "choc:D3_TH_SMD_v2" H 7700 3050 50  0001 C CNN
 F 3 "" H 7700 3050 50  0001 C CNN
 	1    7700 3050
@@
 F 0 "D10" V 8546 2971 50  0000 R CNN
 F 1 "D" V 8455 2971 50  0000 R CNN
-F 2 "SofleKeyboard-footprint:Diode_SOD123" H 8500 3050 50  0001 C CNN
+F 2 "choc:D3_TH_SMD_v2" H 8500 3050 50  0001 C CNN
 F 3 "" H 8500 3050 50  0001 C CNN
 	1    8500 3050
@@
 F 0 "D11" V 9346 2971 50  0000 R CNN
 F 1 "D" V 9255 2971 50  0000 R CNN
-F 2 "SofleKeyboard-footprint:Diode_SOD123" H 9300 3050 50  0001 C CNN
+F 2 "choc:D3_TH_SMD_v2" H 9300 3050 50  0001 C CNN
 F 3 "" H 9300 3050 50  0001 C CNN
 	1    9300 3050
@@
 F 0 "D12" V 10146 2971 50  0000 R CNN
 F 1 "D" V 10055 2971 50  0000 R CNN
-F 2 "SofleKeyboard-footprint:Diode_SOD123" H 10100 3050 50  0001 C CNN
+F 2 "choc:D3_TH_SMD_v2" H 10100 3050 50  0001 C CNN
 F 3 "" H 10100 3050 50  0001 C CNN
 	1    10100 3050
@@
 F 0 "D13" V 6146 3621 50  0000 R CNN
 F 1 "D" V 6055 3621 50  0000 R CNN
-F 2 "SofleKeyboard-footprint:Diode_SOD123" H 6100 3700 50  0001 C CNN
+F 2 "choc:D3_TH_SMD_v2" H 6100 3700 50  0001 C CNN
 F 3 "" H 6100 3700 50  0001 C CNN
 	1    6100 3700
@@
 F 0 "D14" V 6946 3621 50  0000 R CNN
 F 1 "D" V 6855 3621 50  0000 R CNN
-F 2 "SofleKeyboard-footprint:Diode_SOD123" H 6900 3700 50  0001 C CNN
+F 2 "choc:D3_TH_SMD_v2" H 6900 3700 50  0001 C CNN
 F 3 "" H 6900 3700 50  0001 C CNN
 	1    6900 3700
@@
 F 0 "D15" V 7746 3621 50  0000 R CNN
 F 1 "D" V 7655 3621 50  0000 R CNN
-F 2 "SofleKeyboard-footprint:Diode_SOD123" H 7700 3700 50  0001 C CNN
+F 2 "choc:D3_TH_SMD_v2" H 7700 3700 50  0001 C CNN
 F 3 "" H 7700 3700 50  0001 C CNN
 	1    7700 3700
@@
 F 0 "D16" V 8546 3621 50  0000 R CNN
 F 1 "D" V 8455 3621 50  0000 R CNN
-F 2 "SofleKeyboard-footprint:Diode_SOD123" H 8500 3700 50  0001 C CNN
+F 2 "choc:D3_TH_SMD_v2" H 8500 3700 50  0001 C CNN
 F 3 "" H 8500 3700 50  0001 C CNN
 	1    8500 3700
@@
 F 0 "D17" V 9346 3621 50  0000 R CNN
 F 1 "D" V 9255 3621 50  0000 R CNN
-F 2 "SofleKeyboard-footprint:Diode_SOD123" H 9300 3700 50  0001 C CNN
+F 2 "choc:D3_TH_SMD_v2" H 9300 3700 50  0001 C CNN
 F 3 "" H 9300 3700 50  0001 C CNN
 	1    9300 3700
@@
 F 0 "D18" V 10146 3621 50  0000 R CNN
 F 1 "D" V 10055 3621 50  0000 R CNN
-F 2 "SofleKeyboard-footprint:Diode_SOD123" H 10100 3700 50  0001 C CNN
+F 2 "choc:D3_TH_SMD_v2" H 10100 3700 50  0001 C CNN
 F 3 "" H 10100 3700 50  0001 C CNN
 	1    10100 3700
@@
 F 0 "D19" V 6146 4271 50  0000 R CNN
 F 1 "D" V 6055 4271 50  0000 R CNN
-F 2 "SofleKeyboard-footprint:Diode_SOD123" H 6100 4350 50  0001 C CNN
+F 2 "choc:D3_TH_SMD_v2" H 6100 4350 50  0001 C CNN
 F 3 "" H 6100 4350 50  0001 C CNN
 	1    6100 4350
@@
 F 0 "D20" V 6946 4271 50  0000 R CNN
 F 1 "D" V 6855 4271 50  0000 R CNN
-F 2 "SofleKeyboard-footprint:Diode_SOD123" H 6900 4350 50  0001 C CNN
+F 2 "choc:D3_TH_SMD_v2" H 6900 4350 50  0001 C CNN
 F 3 "" H 6900 4350 50  0001 C CNN
 	1    6900 4350
@@
 F 0 "D21" V 7746 4271 50  0000 R CNN
 F 1 "D" V 7655 4271 50  0000 R CNN
-F 2 "SofleKeyboard-footprint:Diode_SOD123" H 7700 4350 50  0001 C CNN
+F 2 "choc:D3_TH_SMD_v2" H 7700 4350 50  0001 C CNN
 F 3 "" H 7700 4350 50  0001 C CNN
 	1    7700 4350
@@
 F 0 "D22" V 8546 4271 50  0000 R CNN
 F 1 "D" V 8455 4271 50  0000 R CNN
-F 2 "SofleKeyboard-footprint:Diode_SOD123" H 8500 4350 50  0001 C CNN
+F 2 "choc:D3_TH_SMD_v2" H 8500 4350 50  0001 C CNN
 F 3 "" H 8500 4350 50  0001 C CNN
 	1    8500 4350
@@
 F 0 "D23" V 9346 4271 50  0000 R CNN
 F 1 "D" V 9255 4271 50  0000 R CNN
-F 2 "SofleKeyboard-footprint:Diode_SOD123" H 9300 4350 50  0001 C CNN
+F 2 "choc:D3_TH_SMD_v2" H 9300 4350 50  0001 C CNN
 F 3 "" H 9300 4350 50  0001 C CNN
 	1    9300 4350
@@
 F 0 "D24" V 10146 4271 50  0000 R CNN
 F 1 "D" V 10055 4271 50  0000 R CNN
-F 2 "SofleKeyboard-footprint:Diode_SOD123" H 10100 4350 50  0001 C CNN
+F 2 "choc:D3_TH_SMD_v2" H 10100 4350 50  0001 C CNN
 F 3 "" H 10100 4350 50  0001 C CNN
 	1    10100 4350
@@
 F 0 "D26" V 6146 4921 50  0000 R CNN
 F 1 "D" V 6055 4921 50  0000 R CNN
-F 2 "SofleKeyboard-footprint:Diode_SOD123" H 6100 5000 50  0001 C CNN
+F 2 "choc:D3_TH_SMD_v2" H 6100 5000 50  0001 C CNN
 F 3 "" H 6100 5000 50  0001 C CNN
 	1    6100 5000
@@
 F 0 "D27" V 6946 4921 50  0000 R CNN
 F 1 "D" V 6855 4921 50  0000 R CNN
-F 2 "SofleKeyboard-footprint:Diode_SOD123" H 6900 5000 50  0001 C CNN
+F 2 "choc:D3_TH_SMD_v2" H 6900 5000 50  0001 C CNN
 F 3 "" H 6900 5000 50  0001 C CNN
 	1    6900 5000
@@
 F 0 "D28" V 7746 4921 50  0000 R CNN
 F 1 "D" V 7655 4921 50  0000 R CNN
-F 2 "SofleKeyboard-footprint:Diode_SOD123" H 7700 5000 50  0001 C CNN
+F 2 "choc:D3_TH_SMD_v2" H 7700 5000 50  0001 C CNN
 F 3 "" H 7700 5000 50  0001 C CNN
 	1    7700 5000
@@
 F 0 "D29" V 8546 4921 50  0000 R CNN
 F 1 "D" V 8455 4921 50  0000 R CNN
-F 2 "SofleKeyboard-footprint:Diode_SOD123" H 8500 5000 50  0001 C CNN
+F 2 "choc:D3_TH_SMD_v2" H 8500 5000 50  0001 C CNN
 F 3 "" H 8500 5000 50  0001 C CNN
 	1    8500 5000
@@
 F 0 "D30" V 9346 4921 50  0000 R CNN
 F 1 "D" V 9255 4921 50  0000 R CNN
-F 2 "SofleKeyboard-footprint:Diode_SOD123" H 9300 5000 50  0001 C CNN
+F 2 "choc:D3_TH_SMD_v2" H 9300 5000 50  0001 C CNN
 F 3 "" H 9300 5000 50  0001 C CNN
 	1    9300 5000
